File: src/diodes_sim.kicad_sch (KiCad schematic)
At the start: 4 parts

Commit message: Added: rough outline
Parts:
- R5: footprint (none) -> EasyEDA:R0603; symbol Device:R -> EasyEDA:CRCW060310K0FKEC; LCSC Part (none) -> C843841
Connections:
- net at D8.2 (A): no longer R5.2
- net at V1.1: no longer R5.1
Changed lines of the file:
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@@
 	)
 	(symbol
-		(lib_id "Device:R")
+		(lib_id "EasyEDA:CRCW060310K0FKEC")
 		(at 134.62 85.09 90)
 		(unit 1)
@@
 			)
 		)
-		(property "Footprint" ""
+		(property "Footprint" "EasyEDA:R0603"
 			(at 134.62 86.868 90)
 			(effects
@@
 			)
 		)
+		(property "LCSC Part" "C843841"
+			(at 144.78 85.09 0)
+			(effects
+				(font
+					(size 1.27 1.27)
+				)
+				(hide yes)
+			)
+		)
