File: src/driver.kicad_sch (KiCad schematic)
At the start: 18 parts, among them Q1 BC547B, Q2 IRFZ44NSTRLPBF

Commit message: Added: rough outline
Parts:
- removed C3: ${SIM.PARAMS}, Capacitor_THT:C_Radial_D5.0mm_H5.0mm_P2.00mm, symbol Device:C
- removed R2, R3, R4: ${SIM.PARAMS}, EasyEDA:RES-TH_BD4.2-L12.0-P16.00-D0.8, symbol Device:R
- added R2: ${SIM.PARAMS}, EasyEDA:R0603, symbol EasyEDA:CRCW060310K0FKEC
- D4: footprint EasyEDA:DO-201_BD5.3-L9.5-P13.50-D1.4-FD -> EasyEDA:USC_L1.7-W1.3-LS2.5-R-RD; LCSC Part C132974 -> C1974448
- D6, D7: footprint EasyEDA:DO-41_BD2.4-L4.7-P8.70-D0.9-RD -> EasyEDA:SMA_L4.3-W2.6-LS5.2-RD; LCSC Part C53568 -> C47921
- OSC1: footprint EasyEDA:PDIP-8_L9.3-W6.4-P2.54-LS7.9-BL-1 -> EasyEDA:SOIC-8_L4.9-W3.9-P1.27-LS6.0-BL; LCSC Part C512178 -> C145607
- Q1: value BC547B -> BC847BT-7-F; footprint EasyEDA:TO-92-3_L4.9-W3.7-P1.27-L -> EasyEDA:SOT-523-3_L1.6-W0.8-P1.00-LS1.6-BR; symbol EasyEDA:BC547B -> EasyEDA:BC847BT-7-F; LCSC Part C713613 -> C156332
- Q2: footprint EasyEDA:TO-220-3_L10.0-W4.5-P2.54-L -> EasyEDA:TO-263-2_L10.0-W9.1-P5.08-LS15.2-TL; LCSC Part C2586 -> C58228
- R1: footprint EasyEDA:RES-TH_BD4.2-L12.0-P16.00-D0.8 -> EasyEDA:R0603; symbol Device:R -> EasyEDA:CRCW060310K0FKEC; LCSC Part (none) -> C843841
Connections:
- net GND: now also Q1.2 (E), Q2.3 (S); no longer Q1.3 (E)
- net VCC: now also R2.1
- net driver_in: now also R1.2; no longer R1.1
- net at OSC1.2 (IN), TP2.1: now also Q1.3 (C), R2.2; no longer Q1.1 (C)
- new net: Q1.1 (B), R1.1, TP1.1
