File: src/driver_sim.kicad_sch (KiCad schematic)
At the start: 13 parts, among them Q7 BC547B, Q8 IRFZ44N

Commit message: Added: rough outline
Parts:
- D34: footprint EasyEDA:DO-201_BD5.3-L9.5-P13.50-D1.4-FD -> EasyEDA:USC_L1.7-W1.3-LS2.5-R-RD; LCSC Part C132974 -> C1974448
- Q7: value BC547B -> BC847BT-7-F; footprint EasyEDA:TO-92-3_L4.9-W3.7-P1.27-L -> EasyEDA:SOT-523-3_L1.6-W0.8-P1.00-LS1.6-BR; symbol EasyEDA:BC547B -> EasyEDA:BC847BT-7-F; LCSC Part C713613 -> C156332
- R26, R27, R28, R29: footprint (none) -> EasyEDA:R0603; symbol Device:R -> EasyEDA:CRCW060310K0FKEC; LCSC Part (none) -> C843841
Connections:
- net 0: now also Q7.2 (E); no longer Q7.3 (E), R28.2
- net at C10.1, D36.2 (A), Q8.2: no longer R29.2
- net at D35.2 (A), L9.1, V3.1: no longer R27.1
- net at L9.2: no longer R29.1
- net at V2.1: no longer R26.1
- net at R26.2: no longer Q7.2 (B)
- new net: D34.1 (A), Q7.3 (C), Q8.1
- now unconnected: Q7.1 (C), R27.2, R28.1
Changed lines of the file:
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@@
 			)
 		)
-		(property "Sim.Params" "y1=0 y2=3.3 td=5m tr=2n tf=2n tw=10m per=20m np=4"
+		(property "Sim.Params" "y1=0 y2=1 td=2n tr=2n tf=2n tw=50n per=100n"
 			(at 111.76 124.3301 0)
 			(effects
@@
 	)
 	(symbol
-		(lib_id "EasyEDA:BC547B")
+		(lib_id "EasyEDA:BC847BT-7-F")
 		(at 138.43 107.95 0)
 		(unit 1)
@@
 			)
 		)
-		(property "Value" "BC547B"
+		(property "Value" "BC847BT-7-F"
 			(at 139.7 109.2199 0)
 			(effects
@@
 			)
 		)
-		(property "Footprint" "EasyEDA:TO-92-3_L4.9-W3.7-P1.27-L"
+		(property "Footprint" "EasyEDA:SOT-523-3_L1.6-W0.8-P1.00-LS1.6-BR"
 			(at 138.43 120.65 0)
 			(effects
@@
 			)
 		)
-		(property "Datasheet" "https://lcsc.com/product-detail/Transistors-NPN-PNP_LGE-BC547B_C713613.html"
+		(property "Datasheet" "https://lcsc.com/product-detail/Transistors-NPN-PNP_DIODES_BC847BT-7-F_BC847BT-7-F_C156332.html"
 			(at 138.43 123.19 0)
 			(effects
@@
 			)
 		)
-		(property "LCSC Part" "C713613"
+		(property "LCSC Part" "C156332"
 			(at 138.43 125.73 0)
 			(effects
@@
 	)
 	(symbol
-		(lib_id "Device:R")
+		(lib_id "EasyEDA:CRCW060310K0FKEC")
 		(at 120.65 107.95 90)
 		(unit 1)
@@
 			)
 		)
-		(property "Footprint" ""
+		(property "Footprint" "EasyEDA:R0603"
 			(at 120.65 109.728 90)
 			(effects
@@
 					(size 1.27 1.27)
 				)
+			)
+		)
+		(property "LCSC Part" "C843841"
+			(at 130.81 107.95 0)
+			(effects
+				(font
+					(size 1.27 1.27)
+				)
+				(hide yes)
 			)
 		)
@@
 	)
 	(symbol
-		(lib_id "Device:R")
+		(lib_id "EasyEDA:CRCW060310K0FKEC")
 		(at 166.37 83.82 0)
 		(unit 1)
@@
 			)
 		)
-		(property "Footprint" ""
+		(property "Footprint" "EasyEDA:R0603"
 			(at 164.592 83.82 90)
 			(effects
@@
 					(size 1.27 1.27)
 				)
+			)
+		)
+		(property "LCSC Part" "C843841"
+			(at 166.37 93.98 0)
+			(effects
+				(font
+					(size 1.27 1.27)
+				)
+				(hide yes)
 			)
 		)
@@
 	)
 	(symbol
-		(lib_id "Device:R")
+		(lib_id "EasyEDA:CRCW060310K0FKEC")
 		(at 148.59 106.68 0)
 		(unit 1)
@@
 			)
 		)
-		(property "Footprint" ""
+		(property "Footprint" "EasyEDA:R0603"
 			(at 146.812 106.68 90)
 			(effects
@@
 					(size 1.27 1.27)
 				)
+			)
+		)
+		(property "LCSC Part" "C843841"
+			(at 148.59 116.84 0)
+			(effects
+				(font
+					(size 1.27 1.27)
+				)
+				(hide yes)
 			)
 		)
@@
 	)
 	(symbol
-		(lib_id "Device:R")
+		(lib_id "EasyEDA:CRCW060310K0FKEC")
 		(at 138.43 93.98 0)
 		(unit 1)
@@
 			)
 		)
-		(property "Footprint" ""
+		(property "Footprint" "EasyEDA:R0603"
 			(at 136.652 93.98 90)
 			(effects
@@
 					(size 1.27 1.27)
 				)
+			)
+		)
+		(property "LCSC Part" "C843841"
+			(at 138.43 104.14 0)
+			(effects
+				(font
+					(size 1.27 1.27)
+				)
+				(hide yes)
 			)
 		)
@@
 			)
 		)
-		(property "Footprint" "EasyEDA:DO-201_BD5.3-L9.5-P13.50-D1.4-FD"
+		(property "Footprint" "EasyEDA:USC_L1.7-W1.3-LS2.5-R-RD"
 			(at 166.37 107.95 0)
 			(effects
@@
 			)
 		)
-		(property "LCSC Part" "C132974"
+		(property "LCSC Part" "C1974448"
 			(at 171.45 107.95 0)
 			(effects
