File: src/injector_PH_driver.kicad_sch (KiCad schematic)
At the start: 11 parts, among them P4 WJ128V-5.0-2P, P5 WJ128V-5.0-2P, P6 WJ128V-5.0-2P, P7 WJ128V-5.0-2P

Commit message: Added: rough outline
Parts:
- D1, D2, D3: footprint EasyEDA:DO-201_BD5.3-L9.5-P13.50-D1.4-FD -> EasyEDA:USC_L1.7-W1.3-LS2.5-R-RD; LCSC Part C132974 -> C1974448
Changed lines of the file:
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@@
 			)
 		)
-		(property "Footprint" "EasyEDA:DO-201_BD5.3-L9.5-P13.50-D1.4-FD"
+		(property "Footprint" "EasyEDA:USC_L1.7-W1.3-LS2.5-R-RD"
 			(at 180.34 58.42 0)
 			(effects
@@
 			)
 		)
-		(property "LCSC Part" "C132974"
+		(property "LCSC Part" "C1974448"
 			(at 185.42 58.42 0)
 			(effects
@@
 			)
 		)
-		(property "Footprint" "EasyEDA:DO-201_BD5.3-L9.5-P13.50-D1.4-FD"
+		(property "Footprint" "EasyEDA:USC_L1.7-W1.3-LS2.5-R-RD"
 			(at 199.39 44.45 0)
 			(effects
@@
 			)
 		)
-		(property "LCSC Part" "C132974"
+		(property "LCSC Part" "C1974448"
 			(at 204.47 44.45 0)
 			(effects
@@
 			)
 		)
-		(property "Footprint" "EasyEDA:DO-201_BD5.3-L9.5-P13.50-D1.4-FD"
+		(property "Footprint" "EasyEDA:USC_L1.7-W1.3-LS2.5-R-RD"
 			(at 194.31 62.23 0)
 			(effects
@@
 			)
 		)
-		(property "LCSC Part" "C132974"
+		(property "LCSC Part" "C1974448"
 			(at 199.39 62.23 0)
 			(effects
