File: src/injector_sense.kicad_sch (KiCad schematic)
At the start: 10 parts

Commit message: Added: rough outline
Parts:
- D22, D23, D24, D25: footprint EasyEDA:DO-41_BD2.4-L4.7-P8.70-D0.9-RD -> EasyEDA:SMA_L4.3-W2.6-LS5.2-RD; LCSC Part C53568 -> C47921
- L3: footprint Inductor_THT_Wurth_NEW:L_Wurth_WE-TI-1016 -> Inductor_THT_Wurth:L_Wurth_WE-TI-1016
- R17, R18: footprint EasyEDA:RES-TH_BD4.2-L12.0-P16.00-D0.8 -> EasyEDA:R0603; symbol Device:R -> EasyEDA:CRCW060310K0FKEC; LCSC Part (none) -> C843841
- gave numbers to parts that had none: 2
Connections:
- net dummy+: no longer R17.2
- net dummy-: no longer R18.1
- net dummy_output_ttl: no longer R17.1, R18.2
Changed lines of the file:
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@@
 			)
 		)
-		(property "Footprint" "Inductor_THT_Wurth_NEW:L_Wurth_WE-TI-1016"
+		(property "Footprint" "Inductor_THT_Wurth:L_Wurth_WE-TI-1016"
 			(at 154.94 67.31 0)
 			(effects
@@
 		(dnp no)
 		(fields_autoplaced yes)
-		(property "Reference" "U?"
+		(property "Reference" "U1"
 			(at 172.72 67.3099 90)
 			(effects
@@
 			(project "injector_PH_driver"
 				(path "/1233132f-6dc2-4199-ab8a-fcffdcb260a3/8918a2e9-3f6a-4d31-a522-7eb8130788f4"
-					(reference "U?")
+					(reference "U1")
 					(unit 1)
 				)
 				(path "/1233132f-6dc2-4199-ab8a-fcffdcb260a3/9693357c-2e3d-4fed-8d76-1154c536c0d4"
-					(reference "U?")
+					(reference "U2")
 					(unit 1)
 				)
@@
 		(dnp no)
 		(fields_autoplaced yes)
-		(property "Reference" "R?"
+		(property "Reference" "R3"
 			(at 172.72 81.2799 90)
 			(effects
@@
 			(project "injector_PH_driver"
 				(path "/1233132f-6dc2-4199-ab8a-fcffdcb260a3/8918a2e9-3f6a-4d31-a522-7eb8130788f4"
-					(reference "R?")
+					(reference "R3")
 					(unit 1)
 				)
 				(path "/1233132f-6dc2-4199-ab8a-fcffdcb260a3/9693357c-2e3d-4fed-8d76-1154c536c0d4"
-					(reference "R?")
+					(reference "R4")
 					(unit 1)
 				)
@@
 			)
 		)
-		(property "Footprint" "EasyEDA:DO-41_BD2.4-L4.7-P8.70-D0.9-RD"
+		(property "Footprint" "EasyEDA:SMA_L4.3-W2.6-LS5.2-RD"
 			(at 125.73 91.44 0)
 			(effects
@@
 			)
 		)
-		(property "Datasheet" "https://lcsc.com/product-detail/Diodes-General-Purpose_ON_1N4007RLG_1N4007RLG_C53568.html"
+		(property "Datasheet" "https://lcsc.com/product-detail/Diodes-General-Purpose_ON_MRA4007T3G_MRA4007T3G_C47921.html"
 			(at 123.19 91.44 0)
 			(effects
@@
 			)
 		)
-		(property "LCSC Part" "C53568"
+		(property "LCSC Part" "C47921"
 			(at 120.65 91.44 0)
 			(effects
@@
 			)
 		)
-		(property "Footprint" "EasyEDA:DO-41_BD2.4-L4.7-P8.70-D0.9-RD"
+		(property "Footprint" "EasyEDA:SMA_L4.3-W2.6-LS5.2-RD"
 			(at 113.03 91.44 0)
 			(effects
@@
 			)
 		)
-		(property "Datasheet" "https://lcsc.com/product-detail/Diodes-General-Purpose_ON_1N4007RLG_1N4007RLG_C53568.html"
+		(property "Datasheet" "https://lcsc.com/product-detail/Diodes-General-Purpose_ON_MRA4007T3G_MRA4007T3G_C47921.html"
 			(at 110.49 91.44 0)
 			(effects
@@
 			)
 		)
-		(property "LCSC Part" "C53568"
+		(property "LCSC Part" "C47921"
 			(at 107.95 91.44 0)
 			(effects
@@
 			)
 		)
-		(property "Footprint" "EasyEDA:DO-41_BD2.4-L4.7-P8.70-D0.9-RD"
+		(property "Footprint" "EasyEDA:SMA_L4.3-W2.6-LS5.2-RD"
 			(at 134.62 91.44 0)
 			(effects
@@
 			)
 		)
-		(property "Datasheet" "https://lcsc.com/product-detail/Diodes-General-Purpose_ON_1N4007RLG_1N4007RLG_C53568.html"
+		(property "Datasheet" "https://lcsc.com/product-detail/Diodes-General-Purpose_ON_MRA4007T3G_MRA4007T3G_C47921.html"
 			(at 137.16 91.44 0)
 			(effects
@@
 			)
 		)
-		(property "LCSC Part" "C53568"
+		(property "LCSC Part" "C47921"
 			(at 139.7 91.44 0)
 			(effects
@@
 			)
 		)
-		(property "Footprint" "EasyEDA:DO-41_BD2.4-L4.7-P8.70-D0.9-RD"
+		(property "Footprint" "EasyEDA:SMA_L4.3-W2.6-LS5.2-RD"
 			(at 147.32 91.44 0)
 			(effects
@@
 			)
 		)
-		(property "Datasheet" "https://lcsc.com/product-detail/Diodes-General-Purpose_ON_1N4007RLG_1N4007RLG_C53568.html"
+		(property "Datasheet" "https://lcsc.com/product-detail/Diodes-General-Purpose_ON_MRA4007T3G_MRA4007T3G_C47921.html"
 			(at 149.86 91.44 0)
 			(effects
@@
 			)
 		)
-		(property "LCSC Part" "C53568"
+		(property "LCSC Part" "C47921"
 			(at 152.4 91.44 0)
 			(effects
@@
 	)
 	(symbol
-		(lib_id "Device:R")
+		(lib_id "EasyEDA:CRCW060310K0FKEC")
 		(at 152.4 72.39 180)
 		(unit 1)
@@
 			)
 		)
-		(property "Footprint" "EasyEDA:RES-TH_BD4.2-L12.0-P16.00-D0.8"
+		(property "Footprint" "EasyEDA:R0603"
 			(at 154.178 72.39 90)
 			(effects
@@
 				)
 				(justify right)
+				(hide yes)
+			)
+		)
+		(property "LCSC Part" "C843841"
+			(at 152.4 62.23 0)
+			(effects
+				(font
+					(size 1.27 1.27)
+				)
 				(hide yes)
 			)
@@
 	)
 	(symbol
-		(lib_id "Device:R")
+		(lib_id "EasyEDA:CRCW060310K0FKEC")
 		(at 152.4 85.09 180)
 		(unit 1)
@@
 			)
 		)
-		(property "Footprint" "EasyEDA:RES-TH_BD4.2-L12.0-P16.00-D0.8"
+		(property "Footprint" "EasyEDA:R0603"
 			(at 154.178 85.09 90)
 			(effects
@@
 				(hide yes)
 			)
+		)
+		(property "LCSC Part" "C843841"
+			(at 152.4 74.93 0)
+			(effects
+				(font
+					(size 1.27 1.27)
+				)
+				(hide yes)
+			)
