File: src/injector_PH_driver.kicad_pcb (KiCad board)
At the start: 2 copper layers, 45 x 57 mm, 34 parts, among them P4 WJ128V-5.0-2P, P5 WJ128V-5.0-2P, P6 WJ128V-5.0-2P, P7 WJ128V-5.0-2P, Q1 BC847BT-7-F, Q2 IRFZ44NSTRLPBF, Q5 BC847BT-7-F, Q6 IRFZ44NSTRLPBF

Commit message: Added. name and version
Parts:
- removed G***: LOGO, LOGO
- C1, C7: footprint EasyEDA:CAP-TH_L5.0-W2.5-P5.00-D1.0 -> CAP-TH_L5.0-W2.5-P5.00-D1.0
- C2, C8: footprint EasyEDA:CAP-TH_L7.3-W4.5-P5.00-D0.5 -> CAP-TH_L7.3-W4.5-P5.00-D0.5
- D1, D14, D2, D3, D4: footprint EasyEDA:USC_L1.7-W1.3-LS2.5-R-RD -> USC_L1.7-W1.3-LS2.5-R-RD
- D15, D5: footprint EasyEDA:DO-27_BD5.2-L8.9-P12.90-D1.5-RD -> DO-27_BD5.2-L8.9-P12.90-D1.5-RD
- D16, D17, D6, D7: footprint EasyEDA:SMA_L4.3-W2.6-LS5.2-RD -> SMA_L4.3-W2.6-LS5.2-RD
- H1, H2, H3, H4: footprint MountingHole:MountingHole_3.5mm_Pad -> MountingHole_3.5mm_Pad
- OSC1, OSC3: footprint EasyEDA:SOIC-8_L4.9-W3.9-P1.27-LS6.0-BL -> SOIC-8_L4.9-W3.9-P1.27-LS6.0-BL
- P4, P5, P6, P7: footprint EasyEDA:CONN-TH_2P-P5.00_WJ128V-5.0-2P -> CONN-TH_2P-P5.00_WJ128V-5.0-2P
- Q1, Q5: footprint EasyEDA:SOT-523-3_L1.6-W0.8-P1.00-LS1.6-BR -> SOT-523-3_L1.6-W0.8-P1.00-LS1.6-BR
- Q2, Q6: footprint EasyEDA:TO-263-2_L10.0-W9.1-P5.08-LS15.2-TL -> TO-263-2_L10.0-W9.1-P5.08-LS15.2-TL
- R1, R10, R11, R2: footprint EasyEDA:R0603 -> R0603
Other:
- board text added: "+"
- board text added: "+12V"
- board text added: "-"
- board text added: "GND"
- board text added: "IN 1"
- board text added: "IN 2"
- board text added: "Inj. 1"
- board text added: "Inj. 2"
- board text added: "Jose Mendonca"
- board text added: "PH Driver V1.2"
- board text added: "github.com/joseluizmendonca"
- board text removed: "BA Jose Mendonça 35756"
